File: LED-PCB/LED.sch (KiCad schematic (older format))
At the start: 72 parts, among them J1 Conn_01x01, J10 Conn_01x01, J11 Conn_01x01, J12 Conn_01x01, J2 Conn_01x01, J3 Conn_01x01, J4 Conn_01x01, J5 Conn_01x01, J6 Conn_01x01, J7 Conn_01x01, J8 Conn_01x01, J9 Conn_01x01

Commit message: Shared libraries
Parts:
- D1, D10, D11, D12, D13, D14, D15, D16, D17, D18, D19, D2, D20, D21, D22, D23, D24, D25, D26, D27, D28, D29, D3, D30, D31, D32, D33, D34, D35, D36, D37, D38, D39, D4, D40, D41, D42, D43, D44, D45, D46, D47, D48, D49, D5, D50, D51, D52, D53, D54, D6, D7, D8, D9: symbol Library:BXEN-50S-11M-3C -> Lighttable:BXEN-50S-11M-3C
Changed lines of the file:
@@
 $EndComp
 $Comp
-L Library:BXEN-50S-11M-3C D6
+L Lighttable:BXEN-50S-11M-3C D6
 U 1 1 61996F29
 P 3400 4450
@@
 	3400 4000 3400 3950
 $Comp
-L Library:BXEN-50S-11M-3C D1
+L Lighttable:BXEN-50S-11M-3C D1
 U 1 1 61998E36
 P 3400 2700
@@
 $EndComp
 $Comp
-L Library:BXEN-50S-11M-3C D2
+L Lighttable:BXEN-50S-11M-3C D2
 U 1 1 619988FA
 P 3400 3050
@@
 $EndComp
 $Comp
-L Library:BXEN-50S-11M-3C D3
+L Lighttable:BXEN-50S-11M-3C D3
 U 1 1 61998468
 P 3400 3400
@@
 $EndComp
 $Comp
-L Library:BXEN-50S-11M-3C D4
+L Lighttable:BXEN-50S-11M-3C D4
 U 1 1 61997EE5
 P 3400 3750
@@
 $EndComp
 $Comp
-L Library:BXEN-50S-11M-3C D5
+L Lighttable:BXEN-50S-11M-3C D5
 U 1 1 61997885
 P 3400 4100
@@
 	5100 4350 5100 4300
 $Comp
-L Library:BXEN-50S-11M-3C D36
+L Lighttable:BXEN-50S-11M-3C D36
 U 1 1 61A91C02
 P 5100 4450
@@
 	5100 4000 5100 3950
 $Comp
-L Library:BXEN-50S-11M-3C D31
+L Lighttable:BXEN-50S-11M-3C D31
 U 1 1 61A91BB8
 P 5100 2700
@@
 $EndComp
 $Comp
-L Library:BXEN-50S-11M-3C D32
+L Lighttable:BXEN-50S-11M-3C D32
 U 1 1 61A91BAE
 P 5100 3050
@@
 $EndComp
 $Comp
-L Library:BXEN-50S-11M-3C D33
+L Lighttable:BXEN-50S-11M-3C D33
 U 1 1 61A91BA4
 P 5100 3400
@@
 $EndComp
 $Comp
-L Library:BXEN-50S-11M-3C D34
+L Lighttable:BXEN-50S-11M-3C D34
 U 1 1 61A91B9A
 P 5100 3750
@@
 $EndComp
 $Comp
-L Library:BXEN-50S-11M-3C D35
+L Lighttable:BXEN-50S-11M-3C D35
 U 1 1 61A91B7A
 P 5100 4100
@@
 $EndComp
 $Comp
-L Library:BXEN-50S-11M-3C D53
+L Lighttable:BXEN-50S-11M-3C D53
 U 1 1 61A91D0A
 P 6150 4100
@@
 $EndComp
 $Comp
-L Library:BXEN-50S-11M-3C D52
+L Lighttable:BXEN-50S-11M-3C D52
 U 1 1 61A91D14
 P 6150 3750
@@
 $EndComp
 $Comp
-L Library:BXEN-50S-11M-3C D51
+L Lighttable:BXEN-50S-11M-3C D51
 U 1 1 61A91D1E
 P 6150 3400
@@
 $EndComp
 $Comp
-L Library:BXEN-50S-11M-3C D50
+L Lighttable:BXEN-50S-11M-3C D50
 U 1 1 61A91D28
 P 6150 3050
@@
 $EndComp
 $Comp
-L Library:BXEN-50S-11M-3C D49
+L Lighttable:BXEN-50S-11M-3C D49
 U 1 1 61A91D32
 P 6150 2700
@@
 	6150 2550 6150 2600
 $Comp
-L Library:BXEN-50S-11M-3C D54
+L Lighttable:BXEN-50S-11M-3C D54
 U 1 1 61A91D7C
 P 6150 4450
@@
 	5800 4350 5800 4300
 $Comp
-L Library:BXEN-50S-11M-3C D48
+L Lighttable:BXEN-50S-11M-3C D48
 U 1 1 61A91CFE
 P 5800 4450
@@
 	5800 4000 5800 3950
 $Comp
-L Library:BXEN-50S-11M-3C D43
+L Lighttable:BXEN-50S-11M-3C D43
 U 1 1 61A91CB4
 P 5800 2700
@@
 $EndComp
 $Comp
-L Library:BXEN-50S-11M-3C D44
+L Lighttable:BXEN-50S-11M-3C D44
 U 1 1 61A91CAA
 P 5800 3050
@@
 $EndComp
 $Comp
-L Library:BXEN-50S-11M-3C D45
+L Lighttable:BXEN-50S-11M-3C D45
 U 1 1 61A91CA0
 P 5800 3400
@@
 $EndComp
 $Comp
-L Library:BXEN-50S-11M-3C D46
+L Lighttable:BXEN-50S-11M-3C D46
 U 1 1 61A91C96
 P 5800 3750
@@
 $EndComp
 $Comp
-L Library:BXEN-50S-11M-3C D47
+L Lighttable:BXEN-50S-11M-3C D47
 U 1 1 61A91C8C
 P 5800 4100
@@
 	5450 4350 5450 4300
 $Comp
-L Library:BXEN-50S-11M-3C D42
+L Lighttable:BXEN-50S-11M-3C D42
 U 1 1 61A91C80
 P 5450 4450
@@
 	5450 4000 5450 3950
 $Comp
-L Library:BXEN-50S-11M-3C D37
+L Lighttable:BXEN-50S-11M-3C D37
 U 1 1 61A91C36
 P 5450 2700
@@
 $EndComp
 $Comp
-L Library:BXEN-50S-11M-3C D38
+L Lighttable:BXEN-50S-11M-3C D38
 U 1 1 61A91C2C
 P 5450 3050
@@
 $EndComp
 $Comp
-L Library:BXEN-50S-11M-3C D39
+L Lighttable:BXEN-50S-11M-3C D39
 U 1 1 61A91C22
 P 5450 3400
@@
 $EndComp
 $Comp
-L Library:BXEN-50S-11M-3C D40
+L Lighttable:BXEN-50S-11M-3C D40
 U 1 1 61A91C18
 P 5450 3750
@@
 $EndComp
 $Comp
-L Library:BXEN-50S-11M-3C D41
+L Lighttable:BXEN-50S-11M-3C D41
 U 1 1 61A91C0E
 P 5450 4100
@@
 $EndComp
 $Comp
-L Library:BXEN-50S-11M-3C D30
+L Lighttable:BXEN-50S-11M-3C D30
 U 1 1 61AC14E0
 P 4750 4450
@@
 	4750 4000 4750 3950
 $Comp
-L Library:BXEN-50S-11M-3C D25
+L Lighttable:BXEN-50S-11M-3C D25
 U 1 1 61AC1496
 P 4750 2700
@@
 $EndComp
 $Comp
-L Library:BXEN-50S-11M-3C D26
+L Lighttable:BXEN-50S-11M-3C D26
 U 1 1 61AC148C
 P 4750 3050
@@
 $EndComp
 $Comp
-L Library:BXEN-50S-11M-3C D27
+L Lighttable:BXEN-50S-11M-3C D27
 U 1 1 61AC1482
 P 4750 3400
@@
 $EndComp
 $Comp
-L Library:BXEN-50S-11M-3C D28
+L Lighttable:BXEN-50S-11M-3C D28
 U 1 1 61AC1478
 P 4750 3750
@@
 $EndComp
 $Comp
-L Library:BXEN-50S-11M-3C D29
+L Lighttable:BXEN-50S-11M-3C D29
 U 1 1 61AC1458
 P 4750 4100
@@
 $EndComp
 $Comp
-L Library:BXEN-50S-11M-3C D24
+L Lighttable:BXEN-50S-11M-3C D24
 U 1 1 61A6802E
 P 4400 4450
@@
 	4400 4000 4400 3950
 $Comp
-L Library:BXEN-50S-11M-3C D19
+L Lighttable:BXEN-50S-11M-3C D19
 U 1 1 61A67FE4
 P 4400 2700
@@
 $EndComp
 $Comp
-L Library:BXEN-50S-11M-3C D20
+L Lighttable:BXEN-50S-11M-3C D20
 U 1 1 61A67FDA
 P 4400 3050
@@
 $EndComp
 $Comp
-L Library:BXEN-50S-11M-3C D21
+L Lighttable:BXEN-50S-11M-3C D21
 U 1 1 61A67FD0
 P 4400 3400
@@
 $EndComp
 $Comp
-L Library:BXEN-50S-11M-3C D22
+L Lighttable:BXEN-50S-11M-3C D22
 U 1 1 61A67FC6
 P 4400 3750
@@
 $EndComp
 $Comp
-L Library:BXEN-50S-11M-3C D23
+L Lighttable:BXEN-50S-11M-3C D23
 U 1 1 61A67FBC
 P 4400 4100
@@
 $EndComp
 $Comp
-L Library:BXEN-50S-11M-3C D18
+L Lighttable:BXEN-50S-11M-3C D18
 U 1 1 61A67FB0
 P 4050 4450
@@
 	4050 4000 4050 3950
 $Comp
-L Library:BXEN-50S-11M-3C D13
+L Lighttable:BXEN-50S-11M-3C D13
 U 1 1 61A67F66
 P 4050 2700
@@
 $EndComp
 $Comp
-L Library:BXEN-50S-11M-3C D14
+L Lighttable:BXEN-50S-11M-3C D14
 U 1 1 61A67F5C
 P 4050 3050
@@
 $EndComp
 $Comp
-L Library:BXEN-50S-11M-3C D15
+L Lighttable:BXEN-50S-11M-3C D15
 U 1 1 61A67F52
 P 4050 3400
@@
 $EndComp
 $Comp
-L Library:BXEN-50S-11M-3C D16
+L Lighttable:BXEN-50S-11M-3C D16
 U 1 1 61A67F48
 P 4050 3750
@@
 $EndComp
 $Comp
-L Library:BXEN-50S-11M-3C D17
+L Lighttable:BXEN-50S-11M-3C D17
 U 1 1 61A67F28
 P 4050 4100
@@
 $EndComp
 $Comp
-L Library:BXEN-50S-11M-3C D12
+L Lighttable:BXEN-50S-11M-3C D12
 U 1 1 61A5E6CF
 P 3750 4450
@@
 	3750 4000 3750 3950
 $Comp
-L Library:BXEN-50S-11M-3C D7
+L Lighttable:BXEN-50S-11M-3C D7
 U 1 1 61A5E685
 P 3750 2700
@@
 $EndComp
 $Comp
-L Library:BXEN-50S-11M-3C D8
+L Lighttable:BXEN-50S-11M-3C D8
 U 1 1 61A5E623
 P 3750 3050
@@
 $EndComp
 $Comp
-L Library:BXEN-50S-11M-3C D9
+L Lighttable:BXEN-50S-11M-3C D9
 U 1 1 61A5E619
 P 3750 3400
@@
 $EndComp
 $Comp
-L Library:BXEN-50S-11M-3C D10
+L Lighttable:BXEN-50S-11M-3C D10
 U 1 1 61A5E60F
 P 3750 3750
@@
 $EndComp
 $Comp
-L Library:BXEN-50S-11M-3C D11
+L Lighttable:BXEN-50S-11M-3C D11
 U 1 1 61A5E605
 P 3750 4100
