File: PS/PS.kicad_pcb (KiCad board)
At the start: 2 copper layers, 174.8 x 29.2 mm, 53 parts, among them J1 Conn_01x01, J10 Conn_01x01, J11 Conn_01x01, J12 Conn_01x01, J13 Conn_01x01, J14 Conn_01x01, J15 Conn_01x01, J2 Conn_01x01, J3 Conn_01x03, J4 Conn_01x01, J5 Conn_01x01, J6 Conn_01x01, J7 Conn_01x01, J8 Conn_01x01, J9 Conn_01x01, Q1 BCP56, Q10 BC848, Q2 BCP56, Q3 BCP56, Q4 BCP56, Q5 BCP56, Q6 BCP56, Q7 BCP56, Q8 BCP56, Q9 BCP56, U1 LM358, U2 LM358, U3 LM358, U4 LM358, U5 LM358

Commit message: Shared libraries
Parts:
- D56: value BZT52Bxx -> 2.4

Commit message: Incorrect value
Parts:
- R14: value 3k -> 150k

Commit message: Vce saturation voltage is too hight, use MOSFET as a switch
Parts:
- Q10: value BC848 -> 2N7002
- R15: value 10k -> 100
Connections:
- net Net-(J10-Pad1) renamed /C8
- net Net-(J11-Pad1) renamed /C3
- net Net-(J12-Pad1) renamed /C9
- net Net-(J13-Pad1) renamed /C4
- net Net-(J14-Pad1) renamed /C5
- net Net-(J6-Pad1) renamed /C6
- net Net-(J7-Pad1) renamed /C1
- net Net-(J8-Pad1) renamed /C7
- net Net-(J9-Pad1) renamed /C2

Commit message: More fixes (magic smoke happened)
Parts:
- added D2: 10, Diode_SMD:D_SOD-123, F.Cu at (155.2, 96.0)
- added D3: B140-E3, Diode_SMD:D_SMA, F.Cu at (187.5, 101.1)
- R13: renamed from R14; value 150k -> 15k
- R14: renamed from R15; value 100 -> 10k
- moved C5 4.83 mm to (157.2, 100.8), turned to 270 degrees
- renumbered D56 to D1, J6 to J1, J5 to J10, J15 to J11, J1 to J12, J2 to J13, J4 to J14, J3 to J15, J7 to J2, J8 to J3, J9 to J4, J10 to J5, J11 to J6, J12 to J7, J13 to J8, J14 to J9, Q2 to Q1, Q1 to Q2, R2 to R1, R12 to R10, R10 to R11, R13 to R12, R1 to R2, R4 to R3, R3 to R4, R6 to R5, R5 to R6, R8 to R7, R7 to R8, R11 to R9
Connections:
- J12 pad 1: VCC -> /VIN
- J14 pad 1: VCC -> /VIN
- U5 pad 5: /Vsense -> Net-(RV1-Pad2)
- U5 pad 6: Net-(RV1-Pad2) -> /Vsense
Routing:
- net /VIN: track 0.00 -> 37.0 mm
- net /Vref: track 160.0 -> 167.2 mm
- net Net-(D2-Pad1): track 2.19 -> 5.08 mm
- net Net-(R14-Pad2): track 10.5 -> 13.2 mm
- net VCC: track 21.8 -> 24.5 mm, vias 6 -> 7
- net /Vsense: track 22.2 -> 23.6 mm
- net Net-(RV1-Pad2): track 17.2 -> 16.6 mm
- net /C9: vias 29 -> 31
- net /C8: vias 29 -> 35
- net /C7: vias 29 -> 35
- net /C6: vias 29 -> 35
- net /C5: vias 27 -> 30
- net /C4: vias 29 -> 31
- net /C3: vias 22 -> 31
- net /C2: vias 28 -> 34
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Other:
- net class Default: trace_width 0.25 -> 0.5
- net class Power added: clearance 0.2, trace_width 1, via_dia 1.6, via_drill 0.8
- net class PowerIn added: clearance 0.2, trace_width 2.5, via_dia 1.6, via_drill 0.8

Commit message: protect sense input
Parts:
- added D4: 1N4148W, Diode_SMD:D_SOD-123, F.Cu at (154.2, 106.2)
- added R15: 10k, Resistor_SMD:R_0805_2012Metric, F.Cu at (149.1, 106.2)
Connections:
- U5 pad 6: /Vsense -> Net-(D4-Pad1)
Routing:
- net Net-(D4-Pad1): track 0.00 -> 9.47 mm
- net /Vsense: track 23.6 -> 26.9 mm
